File: AR488_ESP32/AR488_ESP32.kicad_pcb (KiCad board)
At the start: 2 copper layers, 81.5 x 63.5 mm, 22 parts, among them J1 GPIB_24, J2 DC_7-12V, J3 SHIELD, Q1 AO3401A, Q2 AO3401A, Q3 MMBT5551L, U1 Heltec_WiFi_Kit_32_V2, U2 SN75160BDW, U3 SN75161BN, U4 MCP23017, U5 AMS1117-5.0

Commit message: feat: update GPIB solder footprint — plated oblong mounting holes, 55mm outline
- Mounting holes: plated through-hole oval (3x1mm drill, 3.6x1.6mm pad)
  with pad numbers 25/26 for OUT_SHIELD net connection
- Courtyard width extended from 52.3mm to 55mm
- PCB and schematic updates from KiCad editor (PWR_FLAGs, F8 sync)

Co-Authored-By: Claude Opus 4.6 <noreply@anthropic.com>
Parts:
- C2: value 10u -> 100n
- C6: value 22u -> 1u
- moved C2 67.3 mm to (151.6, 75.7), turned to -90 degrees
- moved C6 47.6 mm to (107.7, 94.0), turned to 180 degrees
- moved U1 0.82 mm to (170.2, 127.7)
Connections:
- net /DC_7-12V renamed DC_7-12V
- net /LDO_IN renamed LDO_IN
- net /LDO_OUTPUT renamed LDO_OUTPUT
Routing:
- net +5V: track 151.1 -> 147.2 mm
- net GND: track 267.8 -> 270.3 mm, vias 9 -> 7
- net +3V3: track 56.4 -> 58.8 mm
- net /NRFD: track 25.6 -> 26.4 mm
- net /SDA: track 37.4 -> 38.2 mm
- net /SCL: track 34.8 -> 35.7 mm
- net /NDAC: track 25.6 -> 26.4 mm
- net /EOI: track 36.8 -> 37.6 mm
- net /DIO8: track 39.7 -> 40.5 mm
- net /DIO7: track 41.2 -> 42.0 mm
- net /DIO6: track 43.1 -> 43.9 mm
- net /DIO5: track 43.8 -> 44.6 mm
- net /DIO4: track 44.9 -> 45.7 mm
- net /DIO3: track 45.1 -> 45.9 mm
- net /DAV: track 25.6 -> 26.4 mm
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Other:
- board size 81.5 x 63.5 mm -> 82.2 x 63.5 mm

Commit message: feat: PCB layout progress — component placement and editor updates
Co-Authored-By: Claude Opus 4.6 <noreply@anthropic.com>
Parts:
- C2: moved to B.Cu
- moved C2 15.5 mm to (167.1, 74.4), turned to 90 degrees
- moved U2 6.03 mm to (158.6, 75.3), turned to -90 degrees
Routing:
- net /DIO8_B: track 29.4 -> 47.1 mm
- net /DIO7_B: track 26.6 -> 42.8 mm
- net GND: track 270.3 -> 286.1 mm, vias 7 -> 6
- net /DIO5_B: track 20.5 -> 35.5 mm, vias 0 -> 2
- net /DIO8: track 40.5 -> 26.2 mm
- net /DIO3_B: track 24.7 -> 38.9 mm, vias 0 -> 1
- net /DIO6_B: track 24.1 -> 37.9 mm, vias 0 -> 2
- net /DIO4_B: track 28.6 -> 42.1 mm, vias 0 -> 2
- net /DIO2_B: track 23.7 -> 36.3 mm, vias 0 -> 1
- net /DIO7: track 42.0 -> 29.7 mm
- net /DIO1_B: track 20.4 -> 32.2 mm, vias 0 -> 1
- net /DIO6: track 43.9 -> 33.3 mm
- net /TE_DATA: track 21.5 -> 32.0 mm
- net /DIO5: track 44.6 -> 36.4 mm
- net /DIO4: track 45.7 -> 39.6 mm
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- added copper zone on B.Cu, net GND
- added copper zone on F.Cu, net GND
Other:
- board size 82.2 x 63.5 mm -> 86 x 67 mm

Commit message: chore: KiCad editor state updates
Co-Authored-By: Claude Opus 4.6 <noreply@anthropic.com>
Other:
- board text added: "AR-488 ESP32 by José Luu F1FGV 2026 V1.0"
Changed lines of the file:
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@@
 		(layer "Edge.Cuts")
+	)
+	(gr_text "AR-488 ESP32 by José Luu F1FGV 2026 V1.0"
+		(at 129.5 70.5 -0)
+		(layer "B.SilkS")
+		(effects
+			(font
+				(size 1 1)
+				(thickness 0.1)
+			)
+			(justify left bottom mirror)
+		)
 	)
 	(segment
