File: AR488_ESP32/AR488_ESP32.kicad_pcb (KiCad board)
At the start: 2 copper layers, 86 x 67 mm, 22 parts, among them J1 GPIB_24, J2 DC_7-12V, J3 SHIELD, Q1 AO3401A, Q2 AO3401A, Q3 MMBT5551L, U1 Heltec_WiFi_Kit_32_V2, U2 SN75160BDW, U3 SN75161BN, U4 MCP23017, U5 AMS1117-5.0

Commit message: feat: v1.1 — PCB and schematic updates, Elecrow manufacturing v1.1
Co-Authored-By: Claude Opus 4.6 <noreply@anthropic.com>
Parts:
- moved R2 2.63 mm to (109.5, 98.9), turned to 0 degrees
Connections:
- Q2 pad 2: LDO_OUTPUT -> +5V
- Q2 pad 3: +5V -> LDO_OUTPUT
- R2 pad 2: GND -> +5V
Routing:
- net +5V: track 146.5 -> 152.5 mm
- net GND: track 286.1 -> 283.2 mm, vias 6 -> 5
- net LDO_OUTPUT: track 12.8 -> 15.1 mm
- net /Q2_GATE: track 13.1 -> 12.0 mm
Other:
- board text added: "AR-488 ESP32 by José Luu F1FGV 2026 V1.1"
- board text removed: "AR-488 ESP32 by José Luu F1FGV 2026 V1.0"
